File: KiCAD Projects/PDB&IO-Board/_saved_science_pdb_io_brd.sch (KiCad schematic (older format))
At the start: 41 parts, among them P1 PWR_IN, P11 ENCODER_1, P13 LIMIT1_IN, P14 LIMIT2_IN, P15 LIMIT3_IN, P16 ENCODER_3, P17 MOTOR1_PWM, P18 MOTOR2_PWM, P19 MOTOR3_PWM, P2 RPI_HEADER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

Commit message: Main Board Layout Mostly Complete
Still needs power routed, but everything else is pretty much finished
now.
Parts:
- P1: footprint (none) -> .pretty:PHOENIX_1792229
Changed lines of the file:
@@
 F 0 "P1" H 2050 1250 50  0000 C CNN
 F 1 "PWR_IN" V 2150 1100 50  0000 C CNN
-F 2 "" H 2050 1100 50  0001 C CNN
+F 2 ".pretty:PHOENIX_1792229" H 2050 1100 50  0001 C CNN
 F 3 "" H 2050 1100 50  0000 C CNN
 	1    2050 1100
