File: KiCAD Projects/PDB&IO-Board/_saved_science_pdb_io_brd.sch (KiCad schematic (older format))
At the start: 46 parts, among them P1 PWR_IN, P10 MOTOR6_PWM, P11 ENCODER_1, P13 LIMIT1_IN, P14 LIMIT2_IN, P15 LIMIT3_IN, P16 ENCODER_3, P17 MOTOR1_PWM, P18 MOTOR2_PWM, P19 MOTOR3_PWM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

Commit message: Started Fixing Errors
Parts:
- C4: value C -> 100nF
- U1: footprint Housings_DIP:DIP-14_W7.62mm -> Housings_SOIC:SOIC-14_3.9x8.7mm_Pitch1.27mm
- U2: footprint (none) -> Housings_SOIC:SOIC-8_3.9x4.9mm_Pitch1.27mm
