File: KiCAD Projects/PDB&IO-Board/science_pdb_io_brd.kicad_pcb (KiCad board)
At the start: 2 copper layers, 146.1 x 94 mm, 46 parts, among them P1 PWR_IN, P11 ENCODER_1, P13 LIMIT1_IN, P14 LIMIT2_IN, P15 LIMIT3_IN, P16 ENCODER_3, P17 MOTOR1_PWM, P18 MOTOR2_PWM, P19 MOTOR3_PWM, P2 RPI_HEADER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

Commit message: Main Board Ready for Review!
Parts:
- added REF**: Hole-M2.5, .pretty:Hole-M2.5, F.Cu at (178.9, 50.1)
- added REF**: HOLE_M3, hole:HOLE_M3, F.Cu at (179.1, 111.8)
- added REF**: HOLE_M3, hole:HOLE_M3, F.Cu at (40.6, 111.8)
- added REF**: HOLE_M3, hole:HOLE_M3, F.Cu at (40.6, 25.4)
- added REF**: HOLE_M3, hole:HOLE_M3, F.Cu at (179.1, 25.4)
- added REF**: VIA-0.4, .pretty:VIA-0.04, F.Cu at (123.8, 41.3)
- added REF**: Hole-M2.5, .pretty:Hole-M2.5, F.Cu at (178.9, 99.2)
- added REF**: Hole-M2.5, .pretty:Hole-M2.5, F.Cu at (121.0, 99.2)
- added REF**: Hole-M2.5, .pretty:Hole-M2.5, F.Cu at (121.0, 50.1)
- moved C4 19.7 mm to (98.4, 31.8), turned to 90 degrees
Other:
- board text added: "Sci Main Board v1 UW Husky Robotics 2017 Cai B. / Jaden B."
- board text removed: "Sci Main Board v1 UW Husky Robotics Cai B. / Jaden B."
Changed lines of the file:
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@@
 (kicad_pcb (version 4) (host pcbnew 4.0.3-stable)
   (general
-    (links 123)
-    (no_connects 2)
+    (links 126)
+    (no_connects 0)
     (area 36.754999 21.514999 182.955001 115.645001)
     (thickness 1.6)
-    (drawings 91)
-    (tracks 456)
+    (drawings 87)
+    (tracks 455)
     (zones 0)
-    (modules 46)
+    (modules 55)
     (nets 130)
   )
@@
   )
   (module Capacitors_SMD:C_1206_HandSoldering (layer F.Cu)
-    (at 117.475 36.83)
+    (at 98.425 31.75 90)
     (descr "Capacitor SMD 1206, hand soldering")
     (tags "capacitor 1206")
     (attr smd)
-    (fp_text reference C4 (at 4.445 0 90) (layer F.SilkS)
-      (effects (font (size 1 1) (thickness 0.15)))
-    )
-    (fp_text value C (at 0 0) (layer F.Fab)
-      (effects (font (size 1 1) (thickness 0.15)))
-    )
-    (fp_text user %R (at 4.445 0 90) (layer F.Fab)
+    (fp_text reference C4 (at 4.445 0 180) (layer F.SilkS)
+      (effects (font (size 1 1) (thickness 0.15)))
+    )
+    (fp_text value C (at 0 0 90) (layer F.Fab)
+      (effects (font (size 1 1) (thickness 0.15)))
+    )
+    (fp_text user %R (at 4.445 0 180) (layer F.Fab)
       (effects (font (size 1 1) (thickness 0.15)))
     )
@@
     (fp_line (start 3.25 1.05) (end 3.25 -1.05) (layer F.CrtYd) (width 0.05))
     (fp_line (start 3.25 1.05) (end -3.25 1.05) (layer F.CrtYd) (width 0.05))
-    (pad 1 smd rect (at -2 0) (size 2 1.6) (layers F.Cu F.Paste F.Mask)
-      (net 73 +3V3))
-    (pad 2 smd rect (at 2 0) (size 2 1.6) (layers F.Cu F.Paste F.Mask)
+    (pad 1 smd rect (at -2 0 90) (size 2 1.6) (layers F.Cu F.Paste F.Mask)
+      (net 73 +3V3))
+    (pad 2 smd rect (at 2 0 90) (size 2 1.6) (layers F.Cu F.Paste F.Mask)
       (net 69 GNDD))
     (model Capacitors_SMD.3dshapes/C_1206.wrl
@@
       (net 69 GNDD) (zone_connect 2))
   )
+  (module .pretty:VIA-0.04 (layer F.Cu)
+    (at 123.825 41.275)
+    (fp_text reference REF** (at 0 1.143) (layer F.SilkS) hide
+      (effects (font (size 0.25 0.25) (thickness 0.05)))
+    )
+    (fp_text value VIA-0.4 (at 0 -1.143) (layer F.Fab) hide
+      (effects (font (size 0.25 0.25) (thickness 0.05)))
+    )
+    (pad 1 thru_hole circle (at 0 0) (size 1.524 1.524) (drill 1.016) (layers *.Cu)
+      (net 69 GNDD) (zone_connect 2))
+  )
+  (module .pretty:Hole-M2.5 (layer F.Cu)
+    (at 178.95 99.15)
+    (fp_text reference REF** (at 0 2.286) (layer F.SilkS) hide
+      (effects (font (size 0.25 0.25) (thickness 0.05)))
+    )
+    (fp_text value Hole-M2.5 (at 0 -2.159) (layer F.Fab) hide
+      (effects (font (size 0.25 0.25) (thickness 0.05)))
+    )
+    (pad 2 thru_hole circle (at 0 0) (size 3.5 3.5) (drill 2.75) (layers *.Cu))
+  )
+  (module .pretty:Hole-M2.5 (layer F.Cu)
+    (at 120.95 99.15)
+    (fp_text reference REF** (at 0 2.286) (layer F.SilkS) hide
+      (effects (font (size 0.25 0.25) (thickness 0.05)))
+    )
+    (fp_text value Hole-M2.5 (at 0 -2.159) (layer F.Fab) hide
+      (effects (font (size 0.25 0.25) (thickness 0.05)))
+    )
+    (pad 2 thru_hole circle (at 0 0) (size 3.5 3.5) (drill 2.75) (layers *.Cu))
+  )
+  (module .pretty:Hole-M2.5 (layer F.Cu)
+    (at 120.95 50.15)
+    (fp_text reference REF** (at 0 2.286) (layer F.SilkS) hide
+      (effects (font (size 0.25 0.25) (thickness 0.05)))
+    )
+    (fp_text value Hole-M2.5 (at 0 -2.159) (layer F.Fab) hide
+      (effects (font (size 0.25 0.25) (thickness 0.05)))
+    )
+    (pad 2 thru_hole circle (at 0 0) (size 3.5 3.5) (drill 2.75) (layers *.Cu))
+  )
+  (module .pretty:Hole-M2.5 (layer F.Cu)
+    (at 178.95 50.15)
+    (fp_text reference REF** (at 0 2.286) (layer F.SilkS) hide
+      (effects (font (size 0.25 0.25) (thickness 0.05)))
+    )
+    (fp_text value Hole-M2.5 (at 0 -2.159) (layer F.Fab) hide
+      (effects (font (size 0.25 0.25) (thickness 0.05)))
+    )
+    (pad 2 thru_hole circle (at 0 0) (size 3.5 3.5) (drill 2.75) (layers *.Cu))
+  )
+  (module hole:HOLE_M3 (layer F.Cu)
+    (at 179.07 111.76)
+    (fp_text reference REF** (at -0.127 3.683) (layer F.SilkS) hide
+      (effects (font (size 1 1) (thickness 0.15)))
+    )
+    (fp_text value HOLE_M3 (at 0.127 -3.683) (layer F.Fab)
+      (effects (font (size 1 1) (thickness 0.15)))
+    )
+    (pad 1 thru_hole circle (at 0 0) (size 5 5) (drill 3.1) (layers *.Cu *.Mask))
+  )
+  (module hole:HOLE_M3 (layer F.Cu)
+    (at 40.64 111.76)
+    (fp_text reference REF** (at -0.127 3.683) (layer F.SilkS) hide
+      (effects (font (size 1 1) (thickness 0.15)))
+    )
+    (fp_text value HOLE_M3 (at 0.127 -3.683) (layer F.Fab)
+      (effects (font (size 1 1) (thickness 0.15)))
+    )
+    (pad 1 thru_hole circle (at 0 0) (size 5 5) (drill 3.1) (layers *.Cu *.Mask))
+  )
+  (module hole:HOLE_M3 (layer F.Cu)
+    (at 40.64 25.4)
+    (fp_text reference REF** (at -0.127 3.683) (layer F.SilkS) hide
+      (effects (font (size 1 1) (thickness 0.15)))
+    )
+    (fp_text value HOLE_M3 (at 0.127 -3.683) (layer F.Fab)
+      (effects (font (size 1 1) (thickness 0.15)))
+    )
+    (pad 1 thru_hole circle (at 0 0) (size 5 5) (drill 3.1) (layers *.Cu *.Mask))
+  )
+  (module hole:HOLE_M3 (layer F.Cu)
+    (at 179.07 25.4)
+    (fp_text reference REF** (at -0.127 3.683) (layer F.SilkS) hide
+      (effects (font (size 1 1) (thickness 0.15)))
+    )
+    (fp_text value HOLE_M3 (at 0.127 -3.683) (layer F.Fab)
+      (effects (font (size 1 1) (thickness 0.15)))
+    )
+    (pad 1 thru_hole circle (at 0 0) (size 5 5) (drill 3.1) (layers *.Cu *.Mask))
+  )
   (gr_text "5V Power" (at 149.225 26.67) (layer B.SilkS)
     (effects (font (size 1 1) (thickness 0.15)) (justify left mirror))
@@
     (effects (font (size 1.5 1.5) (thickness 0.3)) (justify mirror))
   )
-  (gr_text "Sci Main Board v1\nUW Husky Robotics\nCai B. / Jaden B." (at 69.85 105.41) (layer B.SilkS)
+  (gr_text "Sci Main Board v1\nUW Husky Robotics 2017\nCai B. / Jaden B." (at 69.85 105.41) (layer B.SilkS)
     (effects (font (size 1.5 1.5) (thickness 0.3)) (justify mirror))
   )
@@
   (gr_line (start 182.88 21.59) (end 87.63 21.59) (angle 90) (layer Edge.Cuts) (width 0.15))
   (gr_circle (center 178.94 99.145) (end 178.94 102.145) (layer B.SilkS) (width 0.2))
-  (gr_circle (center 178.94 99.145) (end 178.94 100.895) (layer B.SilkS) (width 0.2))
   (gr_circle (center 178.94 50.145) (end 178.94 53.145) (layer B.SilkS) (width 0.2))
-  (gr_circle (center 178.94 50.145) (end 178.94 51.895) (layer B.SilkS) (width 0.2))
-  (gr_circle (center 120.94 99.145) (end 120.94 100.895) (layer B.SilkS) (width 0.2))
   (gr_circle (center 120.94 99.145) (end 120.94 102.145) (layer B.SilkS) (width 0.2))
-  (gr_circle (center 120.94 50.145) (end 120.94 51.895) (layer B.SilkS) (width 0.2))
   (gr_circle (center 120.94 50.145) (end 120.44 53.145) (layer B.SilkS) (width 0.2))
   (gr_line (start 117.44 102.645) (end 117.44 46.645) (angle 90) (layer B.SilkS) (width 0.2))
@@
   (segment (start 142.24 35.56) (end 142.875 35.56) (width 0.508) (layer F.Cu) (net 72))
   (segment (start 142.875 35.56) (end 144.145 35.56) (width 0.508) (layer F.Cu) (net 72))
+  (segment (start 102.87 33.655) (end 98.52 33.655) (width 1.016) (layer F.Cu) (net 73))
+  (segment (start 98.52 33.655) (end 98.425 33.75) (width 1.016) (layer F.Cu) (net 73))
   (segment (start 147.32 35.56) (end 147.955 35.56) (width 0.508) (layer F.Cu) (net 73))
   (segment (start 154.305 36.195) (end 153.67 35.56) (width 0.508) (layer F.Cu) (net 73))
@@
   (segment (start 144.145 33.02) (end 137.795 33.02) (width 1.016) (layer B.Cu) (net 73))
   (segment (start 137.795 33.02) (end 131.445 33.02) (width 1.016) (layer B.Cu) (net 73))
-  (segment (start 115.475 36.83) (end 114.3 36.83) (width 1.016) (layer F.Cu) (net 73))
-  (segment (start 113.03 38.1) (end 111.22 38.1) (width 1.016) (layer F.Cu) (net 73))
-  (segment (start 114.3 36.83) (end 113.03 38.1) (width 1.016) (layer F.Cu) (net 73))
   (segment (start 111.22 38.1) (end 111.22 36.925) (width 1.016) (layer F.Cu) (net 73))
   (segment (start 109.855 35.56) (end 102.87 35.56) (width 1.016) (layer F.Cu) (net 73))

Commit message: Started Fixing Errors
Parts:
- removed the REF** at (178.9, 99.2)
- moved P3 2.54 mm to (44.5, 27.3)
- moved REF** 2.54 mm to (38.1, 111.8)
- moved REF** 2.54 mm to (38.1, 25.4)
Routing:
- net +3V3: track 405.9 -> 408.4 mm
- net /I2C_SDA: track 187.7 -> 190.2 mm
- net /CAM_TRIG: track 154.7 -> 157.3 mm
- net /SPI_DO: track 143.0 -> 145.6 mm
- net /SPI_CLK: track 149.7 -> 152.2 mm
- net /MOTOR3_PWM: track 105.2 -> 107.8 mm
- net GNDA: track 87.7 -> 90.3 mm
- net /SPI_CS: track 154.6 -> 157.2 mm
- net /MOTOR4_PWM: track 104.9 -> 107.4 mm
- net /MOISTURE_IN: track 85.7 -> 88.2 mm
- net /I2C_SCL: track 188.4 -> 191.0 mm
- net +5V: track 282.5 -> 285.1 mm
Other:
- board size 146.1 x 94 mm -> 148.6 x 94 mm
- board text added: "Sci Main Board v1.1 UW Husky Robotics 2017 Cai B. / Jaden B."
- board text removed: "Sci Main Board v1 UW Husky Robotics 2017 Cai B. / Jaden B."

Commit message: Implemented Newest Revisions
Parts:
- added P10: MOTOR6_PWM, Pin_Headers:Pin_Header_Straight_1x03_Pitch2.54mm, B.Cu at (64.8, 101.6)
- added P9: MOTOR5_PWM, Pin_Headers:Pin_Header_Straight_1x03_Pitch2.54mm, B.Cu at (72.4, 101.6)
- added R15: 300Ω, Resistors_SMD:R_1206_HandSoldering, F.Cu at (57.8, 80.6)
- added R18: 300Ω, Resistors_SMD:R_1206_HandSoldering, F.Cu at (54.0, 80.6)
- added REF**: VIA-0.4, .pretty:VIA-0.04, F.Cu at (39.4, 81.9)
- added REF**: VIA-0.4, .pretty:VIA-0.04, F.Cu at (118.1, 43.2)
- added U2: ACPL-064L-500E, Housings_SOIC:SOIC-8_3.9x4.9mm_Pitch1.27mm, F.Cu at (55.9, 90.2)
- C4: value C -> 100nF
- U1: footprint Housings_DIP:DIP-14_W7.62mm -> Housings_SOIC:SOIC-14_3.9x8.7mm_Pitch1.27mm; moved to F.Cu
- moved P21 40.6 mm to (48.3, 109.2)
- moved R2 40.6 mm to (52.7, 102.2)
- moved R1 40.6 mm to (48.9, 102.2)
- moved P20 30.2 mm to (80.0, 101.6), turned to 180 degrees
- moved P19 20.9 mm to (87.6, 101.6), turned to 180 degrees
- moved C4 19.0 mm to (115.6, 40.0), turned to 270 degrees
- moved P18 12.8 mm to (95.2, 101.6), turned to 180 degrees
- moved U1 11.1 mm to (113.0, 30.5)
- moved P17 9.16 mm to (102.9, 101.6), turned to 180 degrees
- moved REF** 3.86 mm to (124.5, 37.5)
Connections:
- P3 pad 21: /SPI_DO -> /MOTOR6_PWM
- P3 pad 42: Net-(P3-Pad42) -> /MOTOR5_PWM
Routing:
- net /SPI_DO: track 145.6 -> 0.00 mm
- net /MOTOR6_PWM: track 0.00 -> 111.5 mm
- net /MOISTURE_IN: track 88.2 -> 33.2 mm
- net +5V: track 285.1 -> 337.9 mm, vias 2 -> 1
- net GNDA: track 90.3 -> 47.9 mm
- net /MOTOR5_PWM: track 0.00 -> 37.8 mm, vias 0 -> 1
- net Net-(P10-Pad2): track 0.00 -> 25.7 mm
- net Net-(P9-Pad2): track 0.00 -> 25.7 mm
- net /MOTOR4_PWM: track 107.4 -> 90.9 mm
- net /MOTOR3_PWM: track 107.8 -> 122.9 mm
- net /B_LIM3: track 38.9 -> 54.0 mm
- net /LIMIT3_IN: track 33.7 -> 20.9 mm
- net /B_LIM1: track 68.7 -> 58.5 mm
- net /MOTOR1_PWM: track 82.7 -> 74.1 mm
- net +3V3: track 408.4 -> 399.8 mm, vias 2 -> 1
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Other:
- board text added: "LIM 1"
- board text added: "LIM 2"
- board text added: "LIM 3"
- board text added: "MOT1"
- board text added: "MOT2"
- board text added: "MOT3"
- board text added: "MOT4"
- board text added: "MOT5"
- board text added: "MOT6"
- board text removed: "ETH Jack"
- board text removed: "LIMSW 1"
- board text removed: "LIMSW 2"
- board text removed: "LIMSW 3"
- board text removed: "MOT1 PWM"
- board text removed: "MOT2 PWM"
- board text removed: "MOT3 PWM"
- board text removed: "MOT4 PWM"
