File: KiCAD Projects/PDB&IO-Board/science_pdb_io_brd.sch (KiCad schematic (older format))
At the start: 41 parts, among them P1 PWR_IN, P11 ENCODER_1, P13 LIMIT1_IN, P14 LIMIT2_IN, P15 LIMIT3_IN, P16 ENCODER_3, P17 MOTOR1_PWM, P18 MOTOR2_PWM, P19 MOTOR3_PWM, P2 RPI_HEADER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

Commit message: Had to change PWM channels
Connections:
- net MOTOR3_PWM: now also P3.16 (P16); no longer P4.45 (P45)
- net MOTOR4_PWM: now also P3.14 (P14); no longer P4.46 (P46)
Changed lines of the file:
@@
 Connection ~ 7650 5800
 Wire Wire Line
-	7200 5800 7750 5800
+	7200 5800 7650 5800
+Wire Wire Line
+	7650 5800 7750 5800
 Wire Wire Line
 	8050 5900 8050 6100
@@
 	5800 5700 5950 5700
 Wire Wire Line
-	5800 5700 5800 7550
+	5800 5700 5800 6250
+Wire Wire Line
+	5800 6250 5800 6800
+Wire Wire Line
+	5800 6800 5800 7350
+Wire Wire Line
+	5800 7350 5800 7550
 Wire Wire Line
 	5900 7150 5950 7150
 Wire Wire Line
-	5900 5250 5900 7150
-Wire Wire Line
-	3300 6200 4550 6200
-Wire Wire Line
-	3300 7100 4550 7100
+	5900 5250 5900 5500
+Wire Wire Line
+	5900 5500 5900 6050
+Wire Wire Line
+	5900 6050 5900 6600
+Wire Wire Line
+	5900 6600 5900 7150
+Wire Wire Line
+	3300 6200 3800 6200
+Wire Wire Line
+	3800 6200 4550 6200
+Wire Wire Line
+	3300 7100 3800 7100
+Wire Wire Line
+	3800 7100 4550 7100
 Connection ~ 4400 7200
 Wire Wire Line
@@
 	4500 7000 4550 7000
 Wire Wire Line
-	4500 6000 4500 7000
+	4500 6000 4500 6100
+Wire Wire Line
+	4500 6100 4500 6550
+Wire Wire Line
+	4500 6550 4500 7000
 Wire Wire Line
 	4400 6300 4550 6300
 Wire Wire Line
-	4400 6300 4400 7300
+	4400 6300 4400 6750
+Wire Wire Line
+	4400 6750 4400 7200
+Wire Wire Line
+	4400 7200 4400 7300
 Wire Wire Line
 	8950 5850 8950 6250
@@
 	1450 6950 1850 6950
 Wire Wire Line
-	2600 6450 2800 6450
+	2600 6450 2700 6450
+Wire Wire Line
+	2700 6450 2800 6450
 Wire Wire Line
 	2700 6450 2700 6350
@@
 Connection ~ 3800 6200
 Wire Wire Line
-	3800 6500 3800 6800
-Wire Wire Line
-	3800 6950 3800 7250
+	3800 6500 3800 6650
+Wire Wire Line
+	3800 6650 3800 6800
+Wire Wire Line
+	3800 6950 3800 7100
+Wire Wire Line
+	3800 7100 3800 7250
 Connection ~ 3800 7100
 Wire Notes Line
@@
 	4150 6800 4100 6800
 Wire Wire Line
-	3300 6650 4550 6650
+	3300 6650 3800 6650
+Wire Wire Line
+	3800 6650 4550 6650
 Connection ~ 3800 6650
 Wire Wire Line
-	3800 6050 3800 6350
+	3800 6050 3800 6200
+Wire Wire Line
+	3800 6200 3800 6350
 Wire Wire Line
 	4150 6400 4150 6350
@@
 	8650 5950 9000 5950
 Wire Wire Line
-	8150 3000 8150 3150
+	8150 3000 8150 3100
+Wire Wire Line
+	8150 3100 8150 3150
 Wire Wire Line
 	8150 3100 8350 3100
@@
 	8850 3100 9050 3100
 Wire Wire Line
-	9050 3000 9050 3150
+	9050 3000 9050 3100
+Wire Wire Line
+	9050 3100 9050 3150
 Wire Wire Line
 	8350 3000 8150 3000
@@
 	7200 4750 7200 4800
 Wire Wire Line
-	6200 4450 7300 4450
-Wire Wire Line
-	6200 4550 7300 4550
-Wire Wire Line
-	6200 4650 7300 4650
+	6200 4450 7000 4450
+Wire Wire Line
+	7000 4450 7300 4450
+Wire Wire Line
+	6200 4550 6800 4550
+Wire Wire Line
+	6800 4550 7300 4550
+Wire Wire Line
+	6200 4650 6600 4650
+Wire Wire Line
+	6600 4650 7300 4650
 Wire Wire Line
 	6600 4400 6600 4650
@@
 	10700 4700 10700 4800
 Wire Wire Line
-	9650 4400 10800 4400
-Wire Wire Line
-	9650 4500 10800 4500
-Wire Wire Line
-	9650 4600 10800 4600
+	9650 4400 10500 4400
+Wire Wire Line
+	10500 4400 10800 4400
+Wire Wire Line
+	9650 4500 10300 4500
+Wire Wire Line
+	10300 4500 10800 4500
+Wire Wire Line
+	9650 4600 10100 4600
+Wire Wire Line
+	10100 4600 10800 4600
 Wire Wire Line
 	10100 4350 10100 4600
@@
 Connection ~ 10300 4500
 Wire Wire Line
-	10300 3950 10300 4050
+	10300 3950 10300 4000
+Wire Wire Line
+	10300 4000 10300 4050
 Wire Wire Line
 	9000 4300 9100 4300
@@
 	9000 4700 9000 4800
 Wire Wire Line
-	7950 4400 9100 4400
-Wire Wire Line
-	7950 4600 9100 4600
+	7950 4400 8800 4400
+Wire Wire Line
+	8800 4400 9100 4400
+Wire Wire Line
+	7950 4600 8400 4600
+Wire Wire Line
+	8400 4600 9100 4600
 Wire Wire Line
 	8400 4350 8400 4600
@@
 	6600 4050 6600 4100
 Wire Wire Line
-	6600 4050 7000 4050
-Wire Wire Line
-	6800 3950 6800 4100
+	6600 4050 6800 4050
+Wire Wire Line
+	6800 4050 7000 4050
+Wire Wire Line
+	6800 3950 6800 4050
+Wire Wire Line
+	6800 4050 6800 4100
 Wire Wire Line
 	7000 4050 7000 4100
 Connection ~ 6800 4050
 Wire Wire Line
-	10100 4000 10500 4000
+	10100 4000 10300 4000
+Wire Wire Line
+	10300 4000 10500 4000
 Wire Wire Line
 	10500 4000 10500 4050
@@
 $EndComp
 Wire Wire Line
-	8400 4000 8800 4000
+	8400 4000 8600 4000
+Wire Wire Line
+	8600 4000 8800 4000
 Wire Wire Line
 	8800 4000 8800 4050
 Wire Wire Line
-	8600 3950 8600 4050
+	8600 3950 8600 4000
+Wire Wire Line
+	8600 4000 8600 4050
 Connection ~ 8600 4000
 Wire Wire Line
@@
 Connection ~ 7000 4450
 Wire Wire Line
-	7950 4500 9100 4500
+	7950 4500 8600 4500
+Wire Wire Line
+	8600 4500 9100 4500
 Wire Wire Line
 	8800 4350 8800 4400
@@
 Wire Wire Line
 	9500 1800 9950 1800
-Text Label 9500 3100 0    40   ~ 0
-MOTOR3_PWM
-Text Label 10900 3100 2    40   ~ 0
-MOTOR4_PWM
-Wire Wire Line
-	10900 3100 10450 3100
-Wire Wire Line
-	9950 3100 9500 3100
 Text Label 9300 2800 2    40   ~ 0
 MOISTURE_IN
@@
 	7150 1050 7300 1050
 Wire Wire Line
-	7300 900  7300 1150
+	7300 900  7300 1050
+Wire Wire Line
+	7300 1050 7300 1150
 Wire Wire Line
 	7150 1250 7300 1250
@@
 	6650 1450 6500 1450
 Wire Wire Line
-	6500 1450 6500 3100
+	6500 1450 6500 2250
+Wire Wire Line
+	6500 2250 6500 2950
+Wire Wire Line
+	6500 2950 6500 3100
 Wire Wire Line
 	6500 2250 6650 2250
@@
 	7300 2650 7150 2650
 Wire Wire Line
-	7300 1250 7300 3100
+	7300 1250 7300 1650
+Wire Wire Line
+	7300 1650 7300 1950
+Wire Wire Line
+	7300 1950 7300 2650
+Wire Wire Line
+	7300 2650 7300 2850
+Wire Wire Line
+	7300 2850 7300 3100
 Wire Wire Line
 	7150 2850 7300 2850
@@
 Wire Wire Line
 	8050 1600 8350 1600
+Wire Wire Line
+	8850 1500 9300 1500
+Wire Wire Line
+	8850 1600 9300 1600
+Text Label 9300 1600 2    40   ~ 0
+MOTOR3_PWM
+Text Label 9300 1500 2    40   ~ 0
+MOTOR4_PWM
 $EndSCHEMATC

Commit message: Main Board Almost Finished
Needs via stitching between ground planes under BeagleBone, then
everything should be connected and ready to go!
Parts:
- P1: footprint (none) -> .pretty:PHOENIX_1792229
- U1: footprint Housings_SOIC:SOIC-14_3.9x8.7mm_Pitch1.27mm -> Housings_DIP:DIP-14_W7.62mm
Changed lines of the file:
@@
 F 0 "U1" H 2250 7150 60  0000 C CNN
 F 1 "SN74HC14N" H 2250 6350 60  0000 C CNN
-F 2 "Housings_SOIC:SOIC-14_3.9x8.7mm_Pitch1.27mm" H 2400 6700 60  0001 C CNN
+F 2 "Housings_DIP:DIP-14_W7.62mm" H 2400 6700 60  0001 C CNN
 F 3 "" H 2400 6700 60  0001 C CNN
 	1    2250 6750
@@
 Connection ~ 7650 5800
 Wire Wire Line
-	7200 5800 7650 5800
-Wire Wire Line
-	7650 5800 7750 5800
+	7200 5800 7750 5800
 Wire Wire Line
 	8050 5900 8050 6100
@@
 	5800 5700 5950 5700
 Wire Wire Line
-	5800 5700 5800 6250
-Wire Wire Line
-	5800 6250 5800 6800
-Wire Wire Line
-	5800 6800 5800 7350
-Wire Wire Line
-	5800 7350 5800 7550
+	5800 5700 5800 7550
 Wire Wire Line
 	5900 7150 5950 7150
 Wire Wire Line
-	5900 5250 5900 5500
-Wire Wire Line
-	5900 5500 5900 6050
-Wire Wire Line
-	5900 6050 5900 6600
-Wire Wire Line
-	5900 6600 5900 7150
-Wire Wire Line
-	3300 6200 3800 6200
-Wire Wire Line
-	3800 6200 4550 6200
-Wire Wire Line
-	3300 7100 3800 7100
-Wire Wire Line
-	3800 7100 4550 7100
+	5900 5250 5900 7150
+Wire Wire Line
+	3300 6200 4550 6200
+Wire Wire Line
+	3300 7100 4550 7100
 Connection ~ 4400 7200
 Wire Wire Line
@@
 	4500 7000 4550 7000
 Wire Wire Line
-	4500 6000 4500 6100
-Wire Wire Line
-	4500 6100 4500 6550
-Wire Wire Line
-	4500 6550 4500 7000
+	4500 6000 4500 7000
 Wire Wire Line
 	4400 6300 4550 6300
 Wire Wire Line
-	4400 6300 4400 6750
-Wire Wire Line
-	4400 6750 4400 7200
-Wire Wire Line
-	4400 7200 4400 7300
+	4400 6300 4400 7300
 Wire Wire Line
 	8950 5850 8950 6250
@@
 	1450 6950 1850 6950
 Wire Wire Line
-	2600 6450 2700 6450
-Wire Wire Line
-	2700 6450 2800 6450
+	2600 6450 2800 6450
 Wire Wire Line
 	2700 6450 2700 6350
@@
 Connection ~ 3800 6200
 Wire Wire Line
-	3800 6500 3800 6650
-Wire Wire Line
-	3800 6650 3800 6800
-Wire Wire Line
-	3800 6950 3800 7100
-Wire Wire Line
-	3800 7100 3800 7250
+	3800 6500 3800 6800
+Wire Wire Line
+	3800 6950 3800 7250
 Connection ~ 3800 7100
 Wire Notes Line
@@
 	4150 6800 4100 6800
 Wire Wire Line
-	3300 6650 3800 6650
-Wire Wire Line
-	3800 6650 4550 6650
+	3300 6650 4550 6650
 Connection ~ 3800 6650
 Wire Wire Line
-	3800 6050 3800 6200
-Wire Wire Line
-	3800 6200 3800 6350
+	3800 6050 3800 6350
 Wire Wire Line
 	4150 6400 4150 6350
@@
 	8650 5950 9000 5950
 Wire Wire Line
-	8150 3000 8150 3100
-Wire Wire Line
-	8150 3100 8150 3150
+	8150 3000 8150 3150
 Wire Wire Line
 	8150 3100 8350 3100
@@
 	8850 3100 9050 3100
 Wire Wire Line
-	9050 3000 9050 3100
-Wire Wire Line
-	9050 3100 9050 3150
+	9050 3000 9050 3150
 Wire Wire Line
 	8350 3000 8150 3000
@@
 	7200 4750 7200 4800
 Wire Wire Line
-	6200 4450 7000 4450
-Wire Wire Line
-	7000 4450 7300 4450
-Wire Wire Line
-	6200 4550 6800 4550
-Wire Wire Line
-	6800 4550 7300 4550
-Wire Wire Line
-	6200 4650 6600 4650
-Wire Wire Line
-	6600 4650 7300 4650
+	6200 4450 7300 4450
+Wire Wire Line
+	6200 4550 7300 4550
+Wire Wire Line
+	6200 4650 7300 4650
 Wire Wire Line
 	6600 4400 6600 4650
@@
 	10700 4700 10700 4800
 Wire Wire Line
-	9650 4400 10500 4400
-Wire Wire Line
-	10500 4400 10800 4400
-Wire Wire Line
-	9650 4500 10300 4500
-Wire Wire Line
-	10300 4500 10800 4500
-Wire Wire Line
-	9650 4600 10100 4600
-Wire Wire Line
-	10100 4600 10800 4600
+	9650 4400 10800 4400
+Wire Wire Line
+	9650 4500 10800 4500
+Wire Wire Line
+	9650 4600 10800 4600
 Wire Wire Line
 	10100 4350 10100 4600
@@
 Connection ~ 10300 4500
 Wire Wire Line
-	10300 3950 10300 4000
-Wire Wire Line
-	10300 4000 10300 4050
+	10300 3950 10300 4050
 Wire Wire Line
 	9000 4300 9100 4300
@@
 	9000 4700 9000 4800
 Wire Wire Line
-	7950 4400 8800 4400
-Wire Wire Line
-	8800 4400 9100 4400
-Wire Wire Line
-	7950 4600 8400 4600
-Wire Wire Line
-	8400 4600 9100 4600
+	7950 4400 9100 4400
+Wire Wire Line
+	7950 4600 9100 4600
 Wire Wire Line
 	8400 4350 8400 4600
@@
 	6600 4050 6600 4100
 Wire Wire Line
-	6600 4050 6800 4050
-Wire Wire Line
-	6800 4050 7000 4050
-Wire Wire Line
-	6800 3950 6800 4050
-Wire Wire Line
-	6800 4050 6800 4100
+	6600 4050 7000 4050
+Wire Wire Line
+	6800 3950 6800 4100
 Wire Wire Line
 	7000 4050 7000 4100
 Connection ~ 6800 4050
 Wire Wire Line
-	10100 4000 10300 4000
-Wire Wire Line
-	10300 4000 10500 4000
+	10100 4000 10500 4000
 Wire Wire Line
 	10500 4000 10500 4050
@@
 $EndComp
 Wire Wire Line
-	8400 4000 8600 4000
-Wire Wire Line
-	8600 4000 8800 4000
+	8400 4000 8800 4000
 Wire Wire Line
 	8800 4000 8800 4050
 Wire Wire Line
-	8600 3950 8600 4000
-Wire Wire Line
-	8600 4000 8600 4050
+	8600 3950 8600 4050
 Connection ~ 8600 4000
 Wire Wire Line
@@
 Connection ~ 7000 4450
 Wire Wire Line
-	7950 4500 8600 4500
-Wire Wire Line
-	8600 4500 9100 4500
+	7950 4500 9100 4500
 Wire Wire Line
 	8800 4350 8800 4400
@@
 F 0 "P1" H 2050 1250 50  0000 C CNN
 F 1 "PWR_IN" V 2150 1100 50  0000 C CNN
-F 2 "" H 2050 1100 50  0001 C CNN
+F 2 ".pretty:PHOENIX_1792229" H 2050 1100 50  0001 C CNN
 F 3 "" H 2050 1100 50  0000 C CNN
 	1    2050 1100
@@
 	7150 1050 7300 1050
 Wire Wire Line
-	7300 900  7300 1050
-Wire Wire Line
-	7300 1050 7300 1150
+	7300 900  7300 1150
 Wire Wire Line
 	7150 1250 7300 1250
@@
 	6650 1450 6500 1450
 Wire Wire Line
-	6500 1450 6500 2250
-Wire Wire Line
-	6500 2250 6500 2950
-Wire Wire Line
-	6500 2950 6500 3100
+	6500 1450 6500 3100
 Wire Wire Line
 	6500 2250 6650 2250
@@
 	7300 2650 7150 2650
 Wire Wire Line
-	7300 1250 7300 1650
-Wire Wire Line
-	7300 1650 7300 1950
-Wire Wire Line
-	7300 1950 7300 2650
-Wire Wire Line
-	7300 2650 7300 2850
-Wire Wire Line
-	7300 2850 7300 3100
+	7300 1250 7300 3100
 Wire Wire Line
 	7150 2850 7300 2850

Commit message: Added Optocoupler and connections for 2 servos
Parts:
- added P10: MOTOR6_PWM, Pin_Headers:Pin_Header_Straight_1x03_Pitch2.54mm, symbol CONN_01X03
- added P9: MOTOR5_PWM, Pin_Headers:Pin_Header_Straight_1x03_Pitch2.54mm, symbol CONN_01X03
- added R15, R18: 300Ω, Resistors_SMD:R_1206_HandSoldering, symbol R
- added U2: ACPL-064L-500E, symbol ACPL-064L-500E
Connections:
- net +5V: now also P10.1 (P1), P9.1 (P1), U2.8 (Vdd)
- net GNDD: now also P10.3 (P3), P9.3 (P3), U2.2 (CA_1), U2.3 (CA_2), U2.5 (GND)
- net SPI_DO: no longer P3.21 (P21)
- net MOTOR5_PWM: now reaches P3.42 (P42)
- net MOTOR5_PWM: now also R15.2
- new net: R15.1, U2.1 (AN_1)
- new net: R18.1, U2.4 (AN_2)
- new net: P10.2 (P2), U2.6 (OUT_2)
- new net: P9.2 (P2), U2.7 (OUT_1)
- new net MOTOR6_PWM: P3.21 (P21), R18.2
Other:
- moved on the sheet: C1, C2, C3, P13, P14, P15, P17, P18, P19, P20, R3, R4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

Commit message: Started Fixing Errors
Parts:
- C4: value C -> 100nF

Commit message: Added Package info for Optocoupler
Forgot to add this to the last commit.
Parts:
- U1: footprint Housings_DIP:DIP-14_W7.62mm -> Housings_SOIC:SOIC-14_3.9x8.7mm_Pitch1.27mm
- U2: footprint (none) -> Housings_SOIC:SOIC-8_3.9x4.9mm_Pitch1.27mm
Changed lines of the file:
@@
 F 0 "U1" H 2250 7150 60  0000 C CNN
 F 1 "SN74HC14N" H 2250 6350 60  0000 C CNN
-F 2 "Housings_DIP:DIP-14_W7.62mm" H 2400 6700 60  0001 C CNN
+F 2 "Housings_SOIC:SOIC-14_3.9x8.7mm_Pitch1.27mm" H 2400 6700 60  0001 C CNN
 F 3 "" H 2400 6700 60  0001 C CNN
 	1    2250 6750
@@
 F 0 "U2" H 2850 3550 60  0000 C CNN
 F 1 "ACPL-064L-500E" H 2600 4050 60  0000 C CNN
-F 2 "" H 2600 3800 60  0001 C CNN
+F 2 "Housings_SOIC:SOIC-8_3.9x4.9mm_Pitch1.27mm" H 2600 3800 60  0001 C CNN
 F 3 "" H 2600 3800 60  0001 C CNN
 	1    2600 3800

Commit message: Submitting for Review.
Parts:
- R1, R10, R11, R12, R13, R14, R16, R17, R2, R3, R4, R5, R6, R7, R8, R9: footprint Capacitors_SMD:C_1206_HandSoldering -> Resistors_SMD:R_1206_HandSoldering
Changed lines of the file:
@@
 F 0 "R1" V 7980 5800 50  0000 C CNN
 F 1 "1kΩ" V 7900 5800 50  0000 C CNN
-F 2 "Capacitors_SMD:C_1206_HandSoldering" V 7830 5800 50  0001 C CNN
+F 2 "Resistors_SMD:R_1206_HandSoldering" V 7830 5800 50  0001 C CNN
 F 3 "" H 7900 5800 50  0000 C CNN
 	1    7900 5800
@@
 F 0 "R2" V 7730 6050 50  0000 C CNN
 F 1 "560Ω" V 7650 6050 50  0000 C CNN
-F 2 "Capacitors_SMD:C_1206_HandSoldering" V 7580 6050 50  0001 C CNN
+F 2 "Resistors_SMD:R_1206_HandSoldering" V 7580 6050 50  0001 C CNN
 F 3 "" H 7650 6050 50  0000 C CNN
 	1    7650 6050
@@
 F 0 "R3" V 5080 6050 50  0000 C CNN
 F 1 "5kΩ" V 5000 6050 50  0000 C CNN
-F 2 "Capacitors_SMD:C_1206_HandSoldering" V 4930 6050 50  0001 C CNN
+F 2 "Resistors_SMD:R_1206_HandSoldering" V 4930 6050 50  0001 C CNN
 F 3 "" H 5000 6050 50  0000 C CNN
 	1    5000 6050
@@
 F 0 "R4" V 5080 6500 50  0000 C CNN
 F 1 "5kΩ" V 5000 6500 50  0000 C CNN
-F 2 "Capacitors_SMD:C_1206_HandSoldering" V 4930 6500 50  0001 C CNN
+F 2 "Resistors_SMD:R_1206_HandSoldering" V 4930 6500 50  0001 C CNN
 F 3 "" H 5000 6500 50  0000 C CNN
 	1    5000 6500
@@
 F 0 "R5" V 5080 6950 50  0000 C CNN
 F 1 "5kΩ" V 5000 6950 50  0000 C CNN
-F 2 "Capacitors_SMD:C_1206_HandSoldering" V 4930 6950 50  0001 C CNN
+F 2 "Resistors_SMD:R_1206_HandSoldering" V 4930 6950 50  0001 C CNN
 F 3 "" H 5000 6950 50  0000 C CNN
 	1    5000 6950
@@
 F 0 "R11" V 8880 4200 50  0000 C CNN
 F 1 "5kΩ" V 8800 4200 50  0000 C CNN
-F 2 "Capacitors_SMD:C_1206_HandSoldering" V 8730 4200 50  0001 C CNN
+F 2 "Resistors_SMD:R_1206_HandSoldering" V 8730 4200 50  0001 C CNN
 F 3 "" H 8800 4200 50  0000 C CNN
 	1    8800 4200
@@
 F 0 "R10" V 8680 4200 50  0000 C CNN
 F 1 "5kΩ" V 8600 4200 50  0000 C CNN
-F 2 "Capacitors_SMD:C_1206_HandSoldering" V 8530 4200 50  0001 C CNN
+F 2 "Resistors_SMD:R_1206_HandSoldering" V 8530 4200 50  0001 C CNN
 F 3 "" H 8600 4200 50  0000 C CNN
 	1    8600 4200
@@
 F 0 "R9" V 8480 4200 50  0000 C CNN
 F 1 "5kΩ" V 8400 4200 50  0000 C CNN
-F 2 "Capacitors_SMD:C_1206_HandSoldering" V 8330 4200 50  0001 C CNN
+F 2 "Resistors_SMD:R_1206_HandSoldering" V 8330 4200 50  0001 C CNN
 F 3 "" H 8400 4200 50  0000 C CNN
 	1    8400 4200
@@
 F 0 "R12" V 10180 4200 50  0000 C CNN
 F 1 "5kΩ" V 10100 4200 50  0000 C CNN
-F 2 "Capacitors_SMD:C_1206_HandSoldering" V 10030 4200 50  0001 C CNN
+F 2 "Resistors_SMD:R_1206_HandSoldering" V 10030 4200 50  0001 C CNN
 F 3 "" H 10100 4200 50  0000 C CNN
 	1    10100 4200
@@
 F 0 "R13" V 10380 4200 50  0000 C CNN
 F 1 "5kΩ" V 10300 4200 50  0000 C CNN
-F 2 "Capacitors_SMD:C_1206_HandSoldering" V 10230 4200 50  0001 C CNN
+F 2 "Resistors_SMD:R_1206_HandSoldering" V 10230 4200 50  0001 C CNN
 F 3 "" H 10300 4200 50  0000 C CNN
 	1    10300 4200
@@
 F 0 "R14" V 10580 4200 50  0000 C CNN
 F 1 "5kΩ" V 10500 4200 50  0000 C CNN
-F 2 "Capacitors_SMD:C_1206_HandSoldering" V 10430 4200 50  0001 C CNN
+F 2 "Resistors_SMD:R_1206_HandSoldering" V 10430 4200 50  0001 C CNN
 F 3 "" H 10500 4200 50  0000 C CNN
 	1    10500 4200
@@
 F 0 "R6" V 6680 4250 50  0000 C CNN
 F 1 "5kΩ" V 6600 4250 50  0000 C CNN
-F 2 "Capacitors_SMD:C_1206_HandSoldering" V 6530 4250 50  0001 C CNN
+F 2 "Resistors_SMD:R_1206_HandSoldering" V 6530 4250 50  0001 C CNN
 F 3 "" H 6600 4250 50  0000 C CNN
 	1    6600 4250
@@
 F 0 "R7" V 6880 4250 50  0000 C CNN
 F 1 "5kΩ" V 6800 4250 50  0000 C CNN
-F 2 "Capacitors_SMD:C_1206_HandSoldering" V 6730 4250 50  0001 C CNN
+F 2 "Resistors_SMD:R_1206_HandSoldering" V 6730 4250 50  0001 C CNN
 F 3 "" H 6800 4250 50  0000 C CNN
 	1    6800 4250
@@
 F 0 "R8" V 7080 4250 50  0000 C CNN
 F 1 "5kΩ" V 7000 4250 50  0000 C CNN
-F 2 "Capacitors_SMD:C_1206_HandSoldering" V 6930 4250 50  0001 C CNN
+F 2 "Resistors_SMD:R_1206_HandSoldering" V 6930 4250 50  0001 C CNN
 F 3 "" H 7000 4250 50  0000 C CNN
 	1    7000 4250
@@
 F 0 "R16" V 1280 1100 50  0000 C CNN
 F 1 "180Ω" V 1200 1100 50  0000 C CNN
-F 2 "Capacitors_SMD:C_1206_HandSoldering" V 1130 1100 50  0001 C CNN
+F 2 "Resistors_SMD:R_1206_HandSoldering" V 1130 1100 50  0001 C CNN
 F 3 "" H 1200 1100 50  0000 C CNN
 	1    1200 1100
@@
 F 0 "R17" V 1630 1100 50  0000 C CNN
 F 1 "80Ω" V 1550 1100 50  0000 C CNN
-F 2 "Capacitors_SMD:C_1206_HandSoldering" V 1480 1100 50  0001 C CNN
+F 2 "Resistors_SMD:R_1206_HandSoldering" V 1480 1100 50  0001 C CNN
 F 3 "" H 1550 1100 50  0000 C CNN
 	1    1550 1100
