File: KiCAD Projects/PDB-Board/science_pdb_io_brd.sch (KiCad schematic (older format))
At the start: 46 parts, among them P1 PWR_IN, P10 MOTOR6_PWM, P11 ENCODER_1, P13 LIMIT1_IN, P14 LIMIT2_IN, P15 LIMIT3_IN, P16 ENCODER_3, P17 MOTOR1_PWM, P18 MOTOR2_PWM, P19 MOTOR3_PWM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

Commit message: Had to Change Encoder Pins Post-Manufacture
The pins we intended to use do not work due to HDMI/eMMC
Connections:
- net ENC1_A: now also P4.14 (P14); no longer P4.22 (P22)
- net ENC1_B: now also P4.16 (P16); no longer P4.24 (P24)
- net ENC1_BUT: no longer P4.20 (P20)
- net ENC2_A: now also P4.17 (P17); no longer P4.28 (P28)
- net ENC2_B: now also P4.18 (P18); no longer P4.30 (P30)
- net ENC2_BUT: no longer P4.26 (P26)
- net ENC3_A: now also P4.7 (P7); no longer P4.34 (P34)
- net ENC3_B: now also P4.9 (P9); no longer P4.36 (P36)
- net ENC3_BUT: no longer P4.32 (P32)
Changed lines of the file:
@@
 EESchema Schematic File Version 2
+LIBS:science_pdb_io_brd-rescue
 LIBS:power
 LIBS:device
@@
 LIBS:contrib
 LIBS:valves
+LIBS:pdb-io
+LIBS:scienceparts
+LIBS:science_pdb_io_brd-cache
 EELAYER 25 0
 EELAYER END
@@
 	1    0    0    -1
 $EndComp
-Text Label 10850 1900 2    40   ~ 0
+Text Label 10850 1500 2    40   ~ 0
 ENC1_A
-Text Label 10850 2000 2    40   ~ 0
+Text Label 10850 1600 2    40   ~ 0
 ENC1_B
-Text Label 10850 2200 2    40   ~ 0
+Text Label 9500 1700 0    40   ~ 0
 ENC2_A
-Text Label 10850 2300 2    40   ~ 0
+Text Label 10850 1700 2    40   ~ 0
 ENC2_B
-Text Label 10850 2500 2    40   ~ 0
+Text Label 9500 1200 0    40   ~ 0
 ENC3_A
-Text Label 10850 2600 2    40   ~ 0
+Text Label 9500 1300 0    40   ~ 0
 ENC3_B
-Text Label 10850 1800 2    40   ~ 0
-ENC1_BUT
-Text Label 10850 2100 2    40   ~ 0
-ENC2_BUT
-Text Label 10850 2400 2    40   ~ 0
-ENC3_BUT
 $Comp
 L GNDD #PWR048
@@
 	2350 1150 2350 1250
 Wire Wire Line
-	10450 2600 10850 2600
-Wire Wire Line
-	10450 2500 10850 2500
-Wire Wire Line
-	10450 2300 10850 2300
-Wire Wire Line
-	10450 2200 10850 2200
-Wire Wire Line
-	10450 2000 10850 2000
-Wire Wire Line
-	10450 1900 10850 1900
-Wire Wire Line
-	10450 1800 10850 1800
-Wire Wire Line
-	10450 2100 10850 2100
-Wire Wire Line
-	10450 2400 10850 2400
-Wire Wire Line
 	7150 1050 7300 1050
 Wire Wire Line
@@
 Wire Wire Line
 	1650 3600 1200 3600
+Wire Wire Line
+	10850 1700 10450 1700
+Wire Wire Line
+	10450 1600 10850 1600
+Wire Wire Line
+	10850 1500 10450 1500
+Wire Wire Line
+	9950 1700 9500 1700
+Wire Wire Line
+	9950 1300 9500 1300
+Wire Wire Line
+	9500 1200 9950 1200
 $EndSCHEMATC
